File: PCB design files/ModMoPSS - RFID module/rfid.sch (EAGLE design)
At the start: 76 parts, among them IC1 LT1761, IC2 7805_TO252, IC3 EM4095, IC4 EM4095, IC5 LT1761

Commit message: Fix for non functional level shifting
Update to fix non functional level shifting on DMOD and CLK pins
Parts:
- removed TEENSYLC1, TEENSYLC2: TEENSYLC, 000-my_library:TEENSYLC
- added D3: SM4007PL, diode:CGRM4007-G
- added PWR2: 22-05-7028-02, con-molex:22-05-7028-02
- added TEENSY_4.0_1, TEENSY_4.0_2: TEENSY40, 000-my_library:TEENSY40
- ANT1, ANT2: value 53048-02 -> 53261-02; device con-molex:53048-02 -> con-molex:53261-02
Connections:
- net ANT1 renamed N$20
- removed net DMOD: IC3.DMOD_OUT, R1.1, R2.2
- removed net DMOD1: IC4.DMOD_OUT, R8.2, R9.1
- removed net RDY/CLK: IC3.RDY/CLK, R3.1, R4.2
- removed net RDY/CLK1: IC4.RDY/CLK, R10.1, R11.2
- new net N$21: C11.1, D3.C, IC2.VI
- new net N$22: IC4.DMOD_OUT, R8.2
- new net N$23: IC3.RDY/CLK, R4.2
- new net N$24: IC3.DMOD_OUT, R2.2
- new net N$26: IC4.RDY/CLK, R11.2
- net +12V: now also D3.A, PWR2-1.S; no longer C11.1, IC2.VI
- net +5V: now also TEENSY_4.0_1.VIN, TEENSY_4.0_2.VIN; no longer TEENSYLC1.VIN, TEENSYLC2.VIN
- net GND: now also PWR2-2.S, TEENSY_4.0_1.GND, TEENSY_4.0_1.GND@1, TEENSY_4.0_1.GND@2, TEENSY_4.0_2.GND, TEENSY_4.0_2.GND@1, TEENSY_4.0_2.GND@2; no longer TEENSYLC1.GND, TEENSYLC1.GND@1, TEENSYLC1.GND@2, TEENSYLC2.GND, TEENSYLC2.GND@1, TEENSYLC2.GND@2
- net LED1: now also TEENSY_4.0_1.23~A9; no longer TEENSYLC1.23~A9
- net LED2: now also TEENSY_4.0_2.23~A9; no longer TEENSYLC2.23~A9
- net N$10: now also TEENSY_4.0_1.3V3, TEENSY_4.0_1.3V3@1; no longer TEENSYLC1.3V3, TEENSYLC1.3V3@1
- net N$11: now also R9.1, TEENSY_4.0_2.6~; no longer TEENSYLC2.6~
- net N$12: now also R10.1, TEENSY_4.0_2.5~; no longer TEENSYLC2.5*
- net N$15: now also TEENSY_4.0_1.7~; no longer TEENSYLC1.7
- net N$16: now also TEENSY_4.0_2.PROGRAM; no longer TEENSYLC2.PROGRAM
- net N$17: now also TEENSY_4.0_2.3V3, TEENSY_4.0_2.3V3@1; no longer TEENSYLC2.3V3, TEENSYLC2.3V3@1
- net N$2: now also R3.1, TEENSY_4.0_1.5~; no longer TEENSYLC1.5*
- net N$6: now also R1.1, TEENSY_4.0_1.6~; no longer TEENSYLC1.6~
- net N$8: now also TEENSY_4.0_1.PROGRAM; no longer TEENSYLC1.PROGRAM
- net SCL: now also TEENSY_4.0_1.19~A5_SCL, TEENSY_4.0_2.19~A5_SCL; no longer TEENSYLC1.19_A5_SCL, TEENSYLC2.19_A5_SCL
- net SDA: now also TEENSY_4.0_1.18~A4_SDA, TEENSY_4.0_2.18~A4_SDA; no longer TEENSYLC1.18_A4_SDA, TEENSYLC2.18_A4_SDA
- net SHD1: now also TEENSY_4.0_2.7~; no longer TEENSYLC2.7
- net STAT1: now also TEENSY_4.0_1.22~A8; no longer TEENSYLC1.22~A8
- net STAT2: now also TEENSY_4.0_2.22~A8; no longer TEENSYLC2.22~A8
Other:
- moved on the sheet: R11, R2, R4, R8, S1, S2
